File: Atmega328_Coursera/Atmega328_Coursera.kicad_sch (KiCad schematic)
At the start: 25 parts, among them J1 USB_A, J2 Conn_01x12, J3 Conn_01x12, U1 ATmega328P-A, U2 AMS1117, Y1 Crystal

Commit message: New updates and Optimization
Parts:
- removed H5: MountingHole_Pad, MountingHole:MountingHole_3.2mm_M3_Pad_TopBottom, symbol Mechanical:MountingHole_Pad
- J2: footprint Connector_PinSocket_2.54mm:PinSocket_1x10_P2.54mm_Vertical -> Connector_PinSocket_2.54mm:PinSocket_1x12_P2.54mm_Vertical
- J3: footprint Connector_PinSocket_2.54mm:PinSocket_1x10_P2.54mm_Vertical -> Connector_PinHeader_2.54mm:PinHeader_1x12_P2.54mm_Vertical
- renumbered C3 to C1, C6 to C2, C7 to C3, C5 to C4, C4 to C5, C1 to C6, C2 to C7, D2 to D1, D3 to D2, D1 to D3, R2 to R1, R3 to R2, R1 to R3, U2 to U1, U1 to U2
