File: Atmega328_Coursera/Atmega328_Coursera.kicad_pcb (KiCad board)
At the start: 2 copper layers, 58 x 41.5 mm, 25 parts, among them J1 USB_A, J2 Conn_01x12, J3 Conn_01x12, U1 ATmega328P-A, U2 AMS1117, Y1 Crystal

Commit message: New updates and Optimization
Parts:
- removed H5: MountingHole_Pad, MountingHole:MountingHole_3.2mm_M3_Pad_TopBottom
- D3: renamed from D1; footprint LED_SMD:LED_0805_2012Metric -> LED_THT:LED_D3.0mm
- J2: footprint Connector_PinSocket_2.54mm:PinSocket_1x10_P2.54mm_Vertical -> Connector_PinSocket_2.54mm:PinSocket_1x12_P2.54mm_Vertical
- J3: footprint Connector_PinSocket_2.54mm:PinSocket_1x10_P2.54mm_Vertical -> Connector_PinHeader_2.54mm:PinHeader_1x12_P2.54mm_Vertical
- moved C2 7.28 mm to (110.6, 60.3), turned to 90 degrees
- moved U1 5.88 mm to (117.9, 59.8), turned to 0 degrees
- moved C1 5.45 mm to (106.1, 63.7), turned to 0 degrees
- moved D3 4.84 mm to (119.2, 70.3), turned to -90 degrees
- moved J3 3.72 mm to (118.5, 91.2)
- moved C3 1.54 mm to (124.6, 64.0)
- moved R5 0.25 mm to (124.2, 73.0)
- renumbered C3 to C1, C6 to C2, C7 to C3, C5 to C4, C4 to C5, C1 to C6, C2 to C7, D2 to D1, D3 to D2, R2 to R1, R3 to R2, R1 to R3, U2 to U1, U1 to U2
Routing:
- net /PD6: track 0.00 -> 31.1 mm, vias 0 -> 2
- net /PC5: track 0.00 -> 22.8 mm, vias 0 -> 1
- net /PC4: track 0.00 -> 20.4 mm, vias 0 -> 1
- net 5VD: track 79.8 -> 74.3 mm
- net /ADC7: track 14.0 -> 18.2 mm
- net /AREF: track 17.2 -> 20.8 mm
- net /ADC6: track 14.0 -> 17.2 mm
- net /PB4: track 26.8 -> 29.9 mm
- net 3V3D: track 59.5 -> 57.3 mm
- net Net-(D3-A): track 2.30 -> 4.21 mm
- net /PC3: track 18.4 -> 17.2 mm
- net /PC2: track 16.3 -> 15.2 mm
- net /PC1: track 13.7 -> 12.7 mm
- net GNDD: track 23.7 -> 22.8 mm, vias 16 -> 14
- net /PC0: track 12.9 -> 12.2 mm

Commit message: Add Guard Trace
Parts:
- moved R4 1.77 mm to (122.3, 78.3)
- moved R5 1.31 mm to (125.0, 72.0), turned to 90 degrees
- turned D3 to 0 degrees
Routing:
- net GNDD: track 22.8 -> 43.7 mm, vias 14 -> 21
- net 5VD: track 74.3 -> 75.7 mm
- net Net-(D3-A): track 4.21 -> 3.61 mm
